Commit message: Broken Code fixed

File: urdf/four_wheel_bot.xacro (robot description, xacro)
@@ -4,6 +4,6 @@
 <xacro:property name="baselw" value="1"/>
 <xacro:property name="baseh" value="0.25"/>
-<xacro:include filename="$(find robolab_mini_project)/src/urdf/materials.xacro" />
-<xacro:include filename="$(find robolab_mini_project)/src/urdf/macros.xacro" />
+<xacro:include filename="$(find robolab_mini_project)/urdf/materials.xacro" />
+<xacro:include filename="$(find robolab_mini_project)/urdf/macros.xacro" />
   <link name="base_link">
   <pose>0 0 3 0 0 0</pose>
@@ -35,4 +35,4 @@
   <xacro:joint_link joint_name="right_joint_2" child="right_wheel_2" origin_xyz="-0.25 -0.55 0.025"/>
   <xacro:joint_link joint_name="left_joint_1" child="left_wheel_1" origin_xyz="0.25 0.55 0.025"/>
-  <xacro:joint_link joint_name="left_joint_2" child="left_wheel_2" origin_xyz="-0.25 -0.55 0.025"/>
+  <xacro:joint_link joint_name="left_joint_2" child="left_wheel_2" origin_xyz="-0.25 0.55 0.025"/>
 </robot>

File: urdf/macros.xacro (robot description, xacro)
@@ -1,5 +1,4 @@
 <?xml version="1.0"?>
 <robot name="four_wheel_bot" xmlns:xacro = "https://www.ros.org/wiki/xacro">
-  <!-- <xacro:include filename="$(find robolab_mini_project)/src/urdf/materials.xacro" /> -->
     <xacro:macro name='wheel_link' params='link_name'>
         <link name="${link_name}">
@@ -29,9 +28,7 @@
         <joint name="${joint_name}" type="continuous">
             <origin xyz="${origin_xyz}" rpy="0 0 0"/>
-            <parent link="chassis"/>
+            <parent link="base_link"/>
             <child link="${child}"/>
             <axis xyz="0 1 0"/>
-            <limit effort="1000" velocity="1000"/>
-            <joint_properties damping="1.0" friction="1.0"/>
         </joint>
     </xacro:macro>

Commit message: Update four_wheel_bot.xacro

File: urdf/four_wheel_bot.xacro (robot description, xacro)
@@ -4,12 +4,11 @@
 <xacro:property name="baselw" value="1"/>
 <xacro:property name="baseh" value="0.25"/>
-<xacro:include filename="$(find robolab_mini_project)/urdf/materials.xacro" />
-<xacro:include filename="$(find robolab_mini_project)/urdf/macros.xacro" />
+<xacro:include filename="$(find robolab_mini_project)/src/urdf/materials.xacro" />
+<xacro:include filename="$(find robolab_mini_project)/src/urdf/macros.xacro" />
+<xacro:include filename="$(find robolab_mini_project)/src/urdf/four_wheel_bot.gazebo"/>
   <link name="base_link">
   <pose>0 0 3 0 0 0</pose>
     <visual>
-      <material name="orange">
-      	<color rgba="1 0.6 0 1"/>
-      </material>
+      <material name="orange"/>
       <origin xyz="0 0 0" rpy="0 0 0" />
       <geometry>
